Commit message: feat(grasp): MuJoCo 任务层 + 开环抓取与成功率扫描
- 场景：CAD URDF 导入后补位置执行器（armature/damping/kv），第二指补反向
  滑动关节 + 等式约束 q2=q1 还原齿条联动，夹持力限 8N
- 抓取：多起点 IK（pan 网格 + 随机 + 枚举位姿当候选）→ 笛卡尔分步下探 →
  合爪 → 笛卡尔抬升；pregrasp 高度按可达性逐档降
- URDF gripper 下限 0.002 → -0.0276：旧值合到底两指仍隔 31.6mm
- 扫描：尺寸 × 半径 × 方位角 24/24；注入 0–15mm 感知偏移 20/20，
  横向容差远大于反投影 0.72cm 中位误差
- 方位角按臂正前方定义（base 绕 z 转了 -90°），否则 +0.2rad 即撞 pan 限位

File: assets/robots/phantomx_pincher_cad/phantomx_pincher_cad.urdf (robot description, URDF)
Before this commit: robot phantomx_pincher_cad, 8 links, 7 joints
Joints:
- joint gripper_joint: limit lower=0.002 upper=0.032 effort=30 velocity=0.5 -> lower=-0.0276 upper=0.032 effort=30 velocity=0.5

File: assets/robots/phantomx_pincher_cad/phantomx_pincher_cad_keypoints.urdf (robot description, URDF)
Before this commit: robot phantomx_pincher_cad, 17 links, 16 joints
Joints:
- joint gripper_joint: limit lower=0.002 upper=0.032 effort=30 velocity=0.5 -> lower=-0.0276 upper=0.032 effort=30 velocity=0.5
